Commit message: Update Real Robot

File: aubo_description/urdf/aubo_i10.urdf.xacro (robot description, xacro)
@@ -211,5 +211,26 @@
     <limit effort="56.0" lower="-3.04" upper="3.04" velocity="3.1416"/>
   </joint>
-  <link name="world"/>
+  <link name="world">
+    <inertial>
+      <origin xyz="0 0 0" rpy="0 0 0" />
+      <mass value="0.0" /> <!-- Massless world link -->
+      <inertia ixx="0" ixy="0" ixz="0" iyy="0" iyz="0" izz="0" />
+    </inertial>
+    <visual>
+      <origin xyz="0 0 -0.001" rpy="0 0 0" />
+      <geometry>
+        <box size="10 10 0.002" /> <!-- Represents a 10x10m flat plane -->
+      </geometry>
+      <material name="gray">
+        <color rgba="0.5 0.5 0.5 1" />
+      </material>
+    </visual>
+    <collision>
+      <origin xyz="0 0 -0.001" rpy="0 0 0" />
+      <geometry>
+        <box size="10 10 0.002" /> <!-- Matches the visual geometry -->
+      </geometry>
+    </collision>
+  </link>
   <joint name="world_joint" type="fixed">
     <parent link="world"/>

File: aubo_description/urdf/aubo_i5.urdf.xacro (robot description, xacro)
@@ -197,5 +197,26 @@
     <limit effort="56.0" lower="-3.04" upper="3.04" velocity="3.1416"/>
   </joint>
-  <link name="world" />
+  <link name="world">
+    <inertial>
+      <origin xyz="0 0 0" rpy="0 0 0" />
+      <mass value="0.0" /> <!-- Massless world link -->
+      <inertia ixx="0" ixy="0" ixz="0" iyy="0" iyz="0" izz="0" />
+    </inertial>
+    <visual>
+      <origin xyz="0 0 -0.001" rpy="0 0 0" />
+      <geometry>
+        <box size="10 10 0.002" /> <!-- Represents a 10x10m flat plane -->
+      </geometry>
+      <material name="gray">
+        <color rgba="0.5 0.5 0.5 1" />
+      </material>
+    </visual>
+    <collision>
+      <origin xyz="0 0 -0.001" rpy="0 0 0" />
+      <geometry>
+        <box size="10 10 0.002" /> <!-- Matches the visual geometry -->
+      </geometry>
+    </collision>
+  </link>
   <joint name="world_joint" type="fixed">
     <parent link="world" />

File: aubo_description/urdf/aubo_i5_depth_camera.urdf.xacro (robot description, xacro)
@@ -212,35 +212,52 @@
       </material>
     </visual>
-    <collision name="collision_top">
+    <collision>
       <origin xyz="0 -0.02 0.034" rpy="0 0 0" />
       <geometry>
-        <box>
-          <size xyz="0.165 0.040 0.030" rpy="0 0 0"/>
-        </box>
-      </geometry>
-    </collision>
-    <collision name="collision_base">
+        <box size="0.165 0.040 0.030"/>
+      </geometry>
+    </collision>
+    <collision>
       <origin xyz="0 -0.010 0.00725" rpy="0 0 0"/>
       <geometry>
-        <box>
-          <size xyz="0.06 0.060 0.015" rpy="0 0 0"/>
-        </box>
-      </geometry>
-    </collision>
-    </link>
-    <joint name='depth_camera_fixed_joint' type='fixed'>
-      <origin xyz="0 0 0" rpy="-1.5708 0 0" />
-      <parent link="wrist3_Link"/>
-      <child link="depth_camera_link"/>
-      <axis xyz="0 0 1" />
-      <limit effort="12.0" lower="0" upper="0" velocity="0"/>
-    </joint>
+        <box size="0.06 0.060 0.015"/>
+      </geometry>
+    </collision>
+  </link>
+  <joint name='depth_camera_fixed_joint' type='fixed'>
+    <origin xyz="0 0 0" rpy="-1.5708 0 0" />
+    <parent link="wrist3_Link"/>
+    <child link="depth_camera_link"/>
+    <axis xyz="0 0 1" />
+    <limit effort="12.0" lower="0" upper="0" velocity="0"/>
+  </joint>
   <link name="depth_camera_optical_link" />
   <joint name="depth_camera_optical_fixed_joint" type="fixed">
     <parent link="depth_camera_link" />
     <child link = "depth_camera_optical_link" />
-    <origin xyz="0.12 0.0 0.0" rpy="0 0 -1.570796" />
-  </joint>
-  <link name="world" />
+    <origin xyz="0.0 0.0 0.0" rpy="0 0 -1.570796" />
+  </joint>
+  <link name="world">
+    <inertial>
+      <origin xyz="0 0 0" rpy="0 0 0" />
+      <mass value="0.0" /> <!-- Massless world link -->
+      <inertia ixx="0" ixy="0" ixz="0" iyy="0" iyz="0" izz="0" />
+    </inertial>
+    <visual>
+      <origin xyz="0 0 -0.001" rpy="0 0 0" />
+      <geometry>
+        <box size="10 10 0.002" /> <!-- Represents a 10x10m flat plane -->
+      </geometry>
+      <material name="gray">
+        <color rgba="0.5 0.5 0.5 1" />
+      </material>
+    </visual>
+    <collision>
+      <origin xyz="0 0 -0.001" rpy="0 0 0" />
+      <geometry>
+        <box size="10 10 0.002" /> <!-- Matches the visual geometry -->
+      </geometry>
+    </collision>
+  </link>
   <joint name="world_joint" type="fixed">
     <parent link="world" />

File: aubo_i10/config/aubo_i10.ros2_control.xacro (robot description, xacro)
@@ -1,11 +1,21 @@
 <?xml version="1.0"?>
 <robot xmlns:xacro="http://www.ros.org/wiki/xacro">
-    <xacro:macro name="aubo_i10_ros2_control" params="name initial_positions_file">
+    <xacro:macro name="aubo_i10_ros2_control" params="name initial_positions_file use_sim_model">
         <xacro:property name="initial_positions" value="${load_yaml(initial_positions_file)['initial_positions']}"/>
+        <xacro:if value="${use_sim_model}">
+            <gazebo>
+                <plugin filename="ign_ros2_control-system" name="ign_ros2_control::IgnitionROS2ControlPlugin">
+                <parameters>$(find aubo_i10)/config/ros2_controllers.yaml</parameters>
+                </plugin>
+            </gazebo>
+        </xacro:if>
         <ros2_control name="${name}" type="system">
             <hardware>
-                <!-- By default, set up controllers for simulation. This won't work on real hardware -->
-                <!-- plugin>mock_components/GenericSystem</plugin -->
+              <xacro:if value="${use_sim_model}">
                 <plugin>ign_ros2_control/IgnitionSystem</plugin>
+              </xacro:if>
+              <xacro:unless value="${use_sim_model}">
+                <plugin>mock_components/GenericSystem</plugin>
+              </xacro:unless>
             </hardware>
             <joint name="shoulder_joint">

File: aubo_i10/config/aubo_i10.urdf.xacro (robot description, xacro)
@@ -1,4 +1,5 @@
 <?xml version="1.0"?>
 <robot xmlns:xacro="http://www.ros.org/wiki/xacro" name="aubo_i10">
+    <xacro:arg name="use_sim_model" default="true"/>
     <xacro:arg name="initial_positions_file" default="initial_positions.yaml" />
     <!-- Import aubo_i10 urdf file -->
@@ -6,9 +7,4 @@
     <!-- Import control_xacro -->
     <xacro:include filename="aubo_i10.ros2_control.xacro" />
-    <xacro:aubo_i10_ros2_control name="IgnitionSystem" initial_positions_file="$(arg initial_positions_file)"/>
-    <gazebo>
-        <plugin filename="ign_ros2_control-system" name="ign_ros2_control::IgnitionROS2ControlPlugin">
-        <parameters>$(find aubo_i10)/config/ros2_controllers.yaml</parameters>
-        </plugin>
-    </gazebo>
+    <xacro:aubo_i10_ros2_control name="Aubosystem" initial_positions_file="$(arg initial_positions_file)" use_sim_model="$(arg use_sim_model)"/>
 </robot>

File: aubo_i5/config/aubo_i5.ros2_control.xacro (robot description, xacro)
@@ -1,11 +1,21 @@
 <?xml version="1.0"?>
 <robot xmlns:xacro="http://www.ros.org/wiki/xacro">
-    <xacro:macro name="aubo_i5_ros2_control" params="name initial_positions_file">
+    <xacro:macro name="aubo_i5_ros2_control" params="name initial_positions_file use_sim_model">
         <xacro:property name="initial_positions" value="${load_yaml(initial_positions_file)['initial_positions']}"/>
+        <xacro:if value="${use_sim_model}">
+            <gazebo>
+                <plugin filename="ign_ros2_control-system" name="ign_ros2_control::IgnitionROS2ControlPlugin">
+                <parameters>$(find aubo_i5)/config/ros2_controllers.yaml</parameters>
+                </plugin>
+            </gazebo>
+        </xacro:if>
         <ros2_control name="${name}" type="system">
             <hardware>
-                <!-- By default, set up controllers for simulation. This won't work on real hardware -->
-                <!-- plugin>mock_components/GenericSystem</plugin -->
+              <xacro:if value="${use_sim_model}">
                 <plugin>ign_ros2_control/IgnitionSystem</plugin>
+              </xacro:if>
+              <xacro:unless value="${use_sim_model}">
+                <plugin>mock_components/GenericSystem</plugin>
+              </xacro:unless>
             </hardware>
             <joint name="shoulder_joint">

File: aubo_i5/config/aubo_i5.urdf.xacro (robot description, xacro)
@@ -1,14 +1,10 @@
 <?xml version="1.0"?>
 <robot xmlns:xacro="http://www.ros.org/wiki/xacro" name="aubo_i5">
+    <xacro:arg name="use_sim_model" default="true"/>
     <xacro:arg name="initial_positions_file" default="initial_positions.yaml" />
     <!-- Import aubo_i5 urdf file -->
     <xacro:include filename="$(find aubo_description)/urdf/aubo_i5.urdf.xacro" />
     <!-- Import control_xacro -->
-    <xacro:include filename="aubo_i5.ros2_control.xacro" />
-    <xacro:aubo_i5_ros2_control name="IgnitionSystem" initial_positions_file="$(arg initial_positions_file)"/>
-    <gazebo>
-        <plugin filename="ign_ros2_control-system" name="ign_ros2_control::IgnitionROS2ControlPlugin">
-        <parameters>$(find aubo_i5)/config/ros2_controllers.yaml</parameters>
-        </plugin>
-    </gazebo>
+    <xacro:include filename="aubo_i5.ros2_control.xacro"/>
+    <xacro:aubo_i5_ros2_control name="Aubosystem" initial_positions_file="$(arg initial_positions_file)" use_sim_model="$(arg use_sim_model)"/>
 </robot>

File: aubo_i5_depth/config/aubo_i5_depth_camera.ros2_control.xacro (robot description, xacro)
@@ -1,10 +1,59 @@
 <?xml version="1.0"?>
 <robot xmlns:xacro="http://www.ros.org/wiki/xacro">
-    <xacro:macro name="aubo_i5_depth_camera_ros2_control" params="name initial_positions_file">
+    <xacro:macro name="aubo_i5_depth_camera_ros2_control" params="name initial_positions_file use_sim_model">
         <xacro:property name="initial_positions" value="${load_yaml(initial_positions_file)['initial_positions']}"/>
+        <xacro:if value="${use_sim_model}">
+            <gazebo>
+                <plugin filename="ign_ros2_control-system" name="ign_ros2_control::IgnitionROS2ControlPlugin">
+                <parameters>$(find aubo_i5_depth)/config/ros2_controllers.yaml</parameters>
+                </plugin>
+            </gazebo>
+            <gazebo reference="depth_camera_link">
+              <sensor type="depth_camera" name="depth_camera_link">
+                <pose>0.12 0 0 0 0 -1.57</pose>
+                <update_rate>5</update_rate>
+                <topic>depth_camera</topic>
+                <ignition_frame_id>depth_camera_optical_link</ignition_frame_id>
+                <camera>
+                  <horizontal_fov>1.05</horizontal_fov>
+                  <image>
+                    <width>256</width>
+                    <height>256</height>
+                    <format>R_FLOAT32</format>
+                  </image>
+                  <clip>
+                    <near>0.10000000000000001</near>
+                    <far>10</far>
+                  </clip>
+                </camera>
+              </sensor>
+              <sensor name="rgb_camera" type="camera">
+                <pose>0.12 0 0 0 0 -1.57</pose>
+                  <camera>
+                    <horizontal_fov>1.05</horizontal_fov>
+                    <image>
+                      <width>256</width>
+                      <height>256</height>
+                    </image>
+                    <clip>
+                      <near>0.1</near>
+                      <far>100</far>
+                    </clip>
+                  </camera>
+                  <always_on>1</always_on>
+                  <update_rate>30</update_rate>
+                  <visualize>true</visualize>
+                  <topic>rgb_camera</topic>
+                </sensor>
+            </gazebo>
+        </xacro:if>
         <ros2_control name="${name}" type="system">
             <hardware>
-                <!-- By default, set up controllers for simulation. This won't work on real hardware -->
+              <xacro:if value="${use_sim_model}">
                 <plugin>ign_ros2_control/IgnitionSystem</plugin>
+              </xacro:if>
+              <xacro:unless value="${use_sim_model}">
+                <plugin>mock_components/GenericSystem</plugin>
+              </xacro:unless>
             </hardware>
             <joint name="shoulder_joint">

File: aubo_i5_depth/config/aubo_i5_depth_camera.urdf.xacro (robot description, xacro)
@@ -1,4 +1,5 @@
 <?xml version="1.0"?>
 <robot xmlns:xacro="http://www.ros.org/wiki/xacro" name="aubo_i5_depth_camera">
+    <xacro:arg name="use_sim_model" default="true"/>
     <xacro:arg name="initial_positions_file" default="initial_positions.yaml" />
     <!-- Import aubo_i5_depth_camera urdf file -->
@@ -6,76 +7,4 @@
     <!-- Import control_xacro -->
     <xacro:include filename="aubo_i5_depth_camera.ros2_control.xacro" />
-    <xacro:aubo_i5_depth_camera_ros2_control name="IgnitionSystem" initial_positions_file="$(arg initial_positions_file)"/>
-    <gazebo>
-        <plugin filename="ign_ros2_control-system" name="ign_ros2_control::IgnitionROS2ControlPlugin">
-        <parameters>$(find aubo_i5_depth)/config/ros2_controllers.yaml</parameters>
-        </plugin>
-    </gazebo>
-    <gazebo reference="depth_camera_link">
-      <sensor type="depth_camera" name="depth_camera_link">
-        <pose>0.12 0 0 0 0 -1.57</pose>
-        <update_rate>5</update_rate>
-        <topic>depth_camera</topic>
-        <ignition_frame_id>depth_camera_optical_link</ignition_frame_id>
-        <camera>
-          <horizontal_fov>1.05</horizontal_fov>
-          <image>
-            <width>256</width>
-            <height>256</height>
-            <format>R_FLOAT32</format>
-          </image>
-          <clip>
-            <near>0.10000000000000001</near>
-            <far>10</far>
-          </clip>
-        </camera>
-      </sensor>
-      <sensor name="rgb_camera" type="camera">
-        <pose>0.12 0 0 0 0 -1.57</pose>
-          <camera>
-            <horizontal_fov>1.05</horizontal_fov>
-            <image>
-              <width>256</width>
-              <height>256</height>
-            </image>
-            <clip>
-              <near>0.1</near>
-              <far>100</far>
-            </clip>
-          </camera>
-          <always_on>1</always_on>
-          <update_rate>30</update_rate>
-          <visualize>true</visualize>
-          <topic>rgb_camera</topic>
-        </sensor>
-    </gazebo>
-    <!-- Adding the box -->
-    <link name="box_link">
-      <inertial>
-        <origin xyz="0 0 0" rpy="0 0 0"/>
-        <mass value="1.0"/>
-        <inertia ixx="0.01" ixy="0" ixz="0" iyy="0.01" iyz="0" izz="0.01"/>
-      </inertial>
-      <visual>
-        <origin xyz="0 0 0" rpy="0 0 0"/>
-        <geometry>
-          <box size="1 1 1"/>
-        </geometry>
-        <material name="blue">
-          <color rgba="0 0 1 1"/>
-        </material>
-      </visual>
-      <collision>
-        <origin xyz="0 0 0" rpy="0 0 0"/>
-        <geometry>
-          <box size="1 1 2"/>
-        </geometry>
-      </collision>
-    </link>
-    <!-- Adding a joint to attach the box -->
-    <joint name="base_to_box" type="fixed">
-      <parent link="world"/>
-      <child link="box_link"/>
-      <origin xyz="0 -2 0" rpy="0 0 0"/>
-    </joint>
+    <xacro:aubo_i5_depth_camera_ros2_control name="Aubosystem" initial_positions_file="$(arg initial_positions_file)" use_sim_model="$(arg use_sim_model)"/>
 </robot>
